File: ControllerMainV2/ControllerMainV2.kicad_pcb (KiCad board)
At the start: 2 copper layers, 392 x 61.8 mm, 180 parts, among them IC1 1462039-4, IC17 TMUX6112PWR, IC18 TMUX6112PWR, IC19 TMUX6112PWR, IC2 TXU0104PWR, IC20 TMUX6112PWR, IC21 TMUX6112PWR, IC22 1462039-4, IC23 1462039-4, IC24 1462039-4, IC25 1462039-4, IC27 1462039-4, IC3 AD75019JPZ, J1 Conn_01x06, J2 Conn_01x10, J24 Conn_01x02, Q1 2N7002, Q2 2N7002, Q3 2N7002, Q4 2N7002, Q5 2N7002, Q6 2N7002, Q7 EL817S1_A__TU_-F, T1 Lehle_MZ_P, U1 MCP23009-E_SO, U10 TL072, U12 TL072, U13 TL072, U14 MCP23009-E_SO, U15 MCP23009-E_SO, U16 MCP23009-E_SO, U18 TL074, U2 MCP23009-E_SO, U9 TL074

Commit message: Main mostly wired. Push for replacement
Parts:
- removed C1, C2, C28: 100n, Capacitor_SMD:C_1206_3216Metric_Pad1.33x1.80mm_HandSolder
- C_U11, C_U9, R67, R68: moved to B.Cu
- D7, D8: footprint Diode_THT:D_DO-41_SOD81_P10.16mm_Horizontal -> Diode_SMD:D_SOD-123
- moved C_U11 351.5 mm to (392.6, 140.1), turned to 90 degrees
- moved C_U9 298.2 mm to (371.6, 139.1), turned to 90 degrees
- moved C31 278.9 mm to (189.6, 181.6), turned to 90 degrees
- moved R67 228.2 mm to (242.8, 159.4)
- moved R68 217.2 mm to (242.8, 155.6)
- moved D7 73.5 mm to (374.1, 162.9)
- moved D8 66.9 mm to (379.9, 162.9)
- moved R33 15.5 mm to (319.9, 132.6)
- moved R32 15.3 mm to (358.1, 132.9)
- moved C11 8.35 mm to (319.9, 129.1), turned to 180 degrees
- moved C10 8.16 mm to (358.1, 129.1), turned to 0 degrees
Routing:
- net /VSS_15V0: track 88.8 -> 634.4 mm, vias 8 -> 18
- net /VDD_15V0: track 33.1 -> 575.9 mm, vias 2 -> 10
- net /Tuner: track 0.00 -> 384.0 mm, vias 0 -> 2
- net GND: track 466.0 -> 687.5 mm, vias 12 -> 34
- net /Addr6: track 2.90 -> 199.7 mm, vias 0 -> 3
- net /Ctrl1: track 3.29 -> 176.8 mm, vias 0 -> 6
- net /Addr7: track 2.90 -> 175.5 mm, vias 0 -> 5
- net /Ctrl2: track 10.4 -> 167.6 mm, vias 0 -> 6
- net /Ctrl4: track 3.55 -> 133.5 mm, vias 0 -> 6
- net Net-(R12-Pad2): track 0.00 -> 113.7 mm, vias 0 -> 4
- net /SwitchMatrix/In16: track 0.00 -> 107.7 mm, vias 0 -> 1
- net /Ctrl3: track 10.2 -> 113.4 mm, vias 0 -> 2
- net Net-(IC18-Pad7): track 0.00 -> 94.9 mm, vias 0 -> 3
- net /Outputs/Conn_Gnd: track 5.21 -> 97.3 mm, vias 0 -> 3
- net Net-(C31-Pad1): track 148.7 -> 236.1 mm, vias 0 -> 3
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
Commit message: Mixer, controll and supply wiring done. Matrix connections missing
Parts:
- removed C_U11, C_U9: 100n, Capacitor_SMD:C_1206_3216Metric_Pad1.33x1.80mm_HandSolder
- added C1: 100n, Capacitor_SMD:C_1206_3216Metric_Pad1.33x1.80mm_HandSolder, B.Cu at (387.2, 146.9)
- added C2: 100n, Capacitor_SMD:C_1206_3216Metric_Pad1.33x1.80mm_HandSolder, B.Cu at (381.6, 146.9)
- C24, C25, C3, C4, C6, C7, C8, C9, Q6, R1, R10, R11, R12, R13, R14, R19, R20, R22, R23, R24, R25, R30, R31, R4, R6, R62, R9: moved to B.Cu
- IC1, IC17, IC18, IC19, IC2, U1: moved to F.Cu
- moved C26 138.5 mm to (520.7, 145.1), turned to 0 degrees
- moved R66 72.2 mm to (328.4, 129.1), turned to 180 degrees
- moved R22 69.5 mm to (319.5, 167.1)
- moved C6 61.3 mm to (324.6, 168.4), turned to 0 degrees
- moved R40 61.1 mm to (384.9, 164.5), turned to 0 degrees
- moved R1 60.5 mm to (324.6, 171.7), turned to 0 degrees
- moved C15 58.2 mm to (378.9, 160.8), turned to 0 degrees
- moved R26 57.7 mm to (324.6, 168.4), turned to 180 degrees
- moved C8 56.3 mm to (330.4, 155.9), turned to 180 degrees
- moved IC2 55.5 mm to (344.8, 130.9)
- moved R24 55.3 mm to (335.5, 157.2), turned to -90 degrees
- moved R39 54.5 mm to (378.9, 164.5), turned to 0 degrees
- moved C30 53.6 mm to (334.7, 131.5), turned to 0 degrees
- moved R5 53.6 mm to (330.4, 152.4), turned to 0 degrees
- moved U1 53.4 mm to (349.5, 179.4), turned to 180 degrees
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Connections:
- C8 pad 2: Net-(C8-Pad2) -> Net-(U18-Pad10)
- C9 pad 2: Net-(C9-Pad2) -> Net-(U18-Pad12)
- IC19 pad 15: Net-(IC19-Pad15) -> Net-(U9-Pad13)
- IC19 pad 2: Net-(IC19-Pad15) -> Net-(U9-Pad13)
- R28 pad 1: Net-(C8-Pad2) -> Net-(U18-Pad10)
- R29 pad 1: Net-(C9-Pad2) -> Net-(U18-Pad12)
- U18 pad 10: Net-(R3-Pad2) -> Net-(U18-Pad10)
- U18 pad 12: Net-(C7-Pad2) -> Net-(U18-Pad12)
- U18 pad 13: Net-(R3-Pad1) -> Net-(R7-Pad1)
- U18 pad 14: Net-(R3-Pad1) -> Net-(R7-Pad1)
- U18 pad 5: Net-(R1-Pad2) -> Net-(C7-Pad2)
- U18 pad 6: Net-(R9-Pad2) -> Net-(R3-Pad1)
- U18 pad 7: Net-(R9-Pad2) -> Net-(R3-Pad1)
- U18 pad 8: Net-(IC17-Pad15) -> Net-(R5-Pad1)
- U18 pad 9: Net-(IC17-Pad15) -> Net-(R5-Pad1)
- U9 pad 1: Net-(R5-Pad1) -> Net-(R9-Pad2)
- U9 pad 10: Net-(R7-Pad2) -> Net-(R5-Pad2)
- U9 pad 12: Net-(C9-Pad2) -> Net-(R7-Pad2)
- U9 pad 13: Net-(R7-Pad1) -> Net-(U9-Pad13)
- U9 pad 14: Net-(R7-Pad1) -> Net-(U9-Pad13)
- U9 pad 2: Net-(R5-Pad1) -> Net-(R9-Pad2)
- U9 pad 3: Net-(C8-Pad2) -> Net-(R1-Pad2)
- U9 pad 5: Net-(R5-Pad2) -> Net-(R3-Pad2)
- U9 pad 6: Net-(R12-Pad1) -> Net-(IC17-Pad15)
- U9 pad 7: Net-(R12-Pad1) -> Net-(IC17-Pad15)
- U9 pad 8: Net-(IC19-Pad15) -> Net-(R12-Pad1)
- U9 pad 9: Net-(IC19-Pad15) -> Net-(R12-Pad1)
Routing:
- net /in: track 429.1 -> 33.0 mm, vias 2 -> 1
- net /send1: track 377.5 -> 0.00 mm, vias 2 -> 0
- net /return1: track 364.6 -> 0.00 mm, vias 1 -> 0
- net /send2: track 355.1 -> 0.00 mm, vias 2 -> 0
- net /return2: track 339.5 -> 0.00 mm, vias 1 -> 0
- net /send3: track 338.8 -> 0.00 mm, vias 2 -> 0
- net /return3: track 318.3 -> 0.00 mm, vias 1 -> 0
- net /send4: track 312.2 -> 0.00 mm, vias 2 -> 0
- net /return4: track 297.6 -> 0.00 mm, vias 1 -> 0
- net /send5: track 291.5 -> 0.00 mm, vias 2 -> 0
- net /return5: track 277.1 -> 0.00 mm, vias 1 -> 0
- net /send6: track 271.6 -> 0.00 mm, vias 2 -> 0
- net /return6: track 260.2 -> 0.00 mm, vias 2 -> 0
- net /return7: track 247.4 -> 0.00 mm, vias 2 -> 0
- net /send7: track 244.5 -> 0.00 mm, vias 2 -> 0
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- added copper zone on F.Cu, net /VDD_5V0
- removed copper zone on F.Cu, net /VDD_3V3

Commit message: DRC clean PCB
Parts:
- C26: moved to B.Cu
- D2, D3: moved to F.Cu
- moved C26 166.3 mm to (355.1, 130.8)
- moved D3 3.42 mm to (292.6, 142.2)
Routing:
- net /send1: track 0.00 -> 329.8 mm, vias 0 -> 2
- net /in: track 33.0 -> 350.9 mm
- net /send2: track 0.00 -> 307.4 mm, vias 0 -> 2
- net /return1: track 0.00 -> 302.5 mm, vias 0 -> 1
- net /send3: track 0.00 -> 285.4 mm, vias 0 -> 2
- net /return2: track 0.00 -> 280.6 mm
- net /send4: track 0.00 -> 264.3 mm, vias 0 -> 2
- net /return3: track 0.00 -> 259.0 mm
- net /send5: track 0.00 -> 241.2 mm, vias 0 -> 2
- net /return4: track 0.00 -> 236.9 mm
- net /send6: track 0.00 -> 217.9 mm, vias 0 -> 2
- net /return5: track 0.00 -> 214.7 mm
- net /send7: track 0.00 -> 194.5 mm, vias 0 -> 2
- net /return6: track 0.00 -> 193.2 mm
- net /expr1: track 0.00 -> 181.8 mm, vias 0 -> 8
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Other:
- board text added: "Controller Main Rev. 2.0"
- board text removed: "3V3"
- board text removed: "Controller Main Rev. 1.0"
- board text removed: "Ctrl1 Gnd"
- board text removed: "Ctrl2 Gnd"
- board text removed: "Exp1"
- board text removed: "Exp2"
- board text removed: "Gnd"
- board text removed: "R10"
- board text removed: "S6"
- board text removed: "S7"
- board text removed: "S8"
- board text removed: "T1"
- board text removed: "T2"

Commit message: Fixed library imports
Routing:
- net GND: track 595.6 -> 590.0 mm
- net /VDD_15V0: track 678.2 -> 676.0 mm
- net /VSS_15V0: track 651.6 -> 650.0 mm
- net /I2C_Reset: track 425.1 -> 423.7 mm
- net Net-(C31-Pad1): track 273.3 -> 272.0 mm
- net /send4: track 264.3 -> 263.5 mm
- net Net-(R10-Pad2): track 47.6 -> 46.9 mm
- net Net-(R14-Pad2): track 21.9 -> 21.1 mm
- net Net-(R12-Pad2): track 27.3 -> 26.5 mm
- net Net-(R39-Pad1): track 21.7 -> 21.0 mm
- net /return6: track 193.2 -> 192.5 mm
- net /return4: track 236.9 -> 236.2 mm
- net /return2: track 280.6 -> 279.9 mm
- net /return1: track 302.5 -> 301.8 mm
- net /in: track 350.9 -> 350.2 mm
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