File: ControllerMainV2/ControllerMainV2.kicad_pcb (KiCad board)
At the start: 2 copper layers, 392 x 61.8 mm, 177 parts, among them IC1 1462039-4, IC17 TMUX6112PWR, IC18 TMUX6112PWR, IC19 TMUX6112PWR, IC2 TXU0104PWR, IC20 TMUX6112PWR, IC21 TMUX6112PWR, IC22 1462039-4, IC23 1462039-4, IC24 1462039-4, IC25 1462039-4, IC27 1462039-4, IC3 AD75019JPZ, J1 Conn_01x06, J2 Conn_01x10, J24 Conn_01x02, Q1 2N7002, Q2 2N7002, Q3 2N7002, Q4 2N7002, Q5 2N7002, Q6 2N7002, Q7 EL817S1_A__TU_-F, T1 Lehle_MZ_P, U1 MCP23009-E_SO, U10 TL072, U12 TL072, U13 TL072, U14 MCP23009-E_SO, U15 MCP23009-E_SO, U16 MCP23009-E_SO, U18 TL074, U2 MCP23009-E_SO, U9 TL074

Commit message: Added pin header for matrix test
Parts:
- added J3: Conn_02x08_Odd_Even, Connector_PinHeader_1.27mm:PinHeader_2x08_P1.27mm_Vertical_SMD, F.Cu at (314.8, 133.4)
- added J4: Conn_02x08_Odd_Even, Connector_PinHeader_1.27mm:PinHeader_2x08_P1.27mm_Vertical_SMD, F.Cu at (185.2, 133.3)
Routing:
- net /out2: track 48.3 -> 216.9 mm, vias 3 -> 6
- net /SwitchMatrix/Out13: track 33.3 -> 192.1 mm, vias 2 -> 5
- net /SwitchMatrix/Out14: track 28.5 -> 185.0 mm, vias 2 -> 5
- net /SwitchMatrix/Out15: track 15.6 -> 167.0 mm, vias 0 -> 1
- net /SwitchMatrix/Out16: track 19.3 -> 159.7 mm, vias 0 -> 1
- net /out1: track 104.7 -> 210.7 mm, vias 5 -> 6
- net /send10: track 146.5 -> 215.5 mm, vias 2 -> 3
- net /send9: track 164.8 -> 218.2 mm
- net /send8: track 181.6 -> 221.9 mm
- net /send7: track 194.2 -> 232.3 mm
- net /SwitchMatrix/In15: track 9.74 -> 46.1 mm
- net /send6: track 217.9 -> 253.4 mm
- net /SwitchMatrix/In16: track 29.8 -> 64.3 mm
- net /send5: track 241.2 -> 274.0 mm
- net /send4: track 263.5 -> 294.0 mm
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
Commit message: 3D models and fixed pcbs
Parts:
- removed J24: Conn_01x02, Connector_PinSocket_2.54mm:PinSocket_1x02_P2.54mm_Vertical
- IC3: footprint Package_LCC:PLCC-44_SMD-Socket -> SamacSys_Parts:69802144LF
- PS1: moved to F.Cu
- moved PS1 7.55 mm to (203.3, 181.5), turned to 180 degrees
- moved J2 6.18 mm to (401.6, 160.1)
- moved J1 5.50 mm to (401.6, 176.1)
- moved H2 0.75 mm to (398.3, 182.9)
- moved R7 0.60 mm to (324.7, 153.0)
- moved H1 0.37 mm to (398.3, 130.9)
Routing:
- net /in: track 372.7 -> 358.7 mm
- net /out2: track 216.9 -> 225.0 mm
- net /CS: track 91.5 -> 99.4 mm
- net /EN_SPL: track 33.4 -> 40.8 mm
- net /VSS_15V0: track 650.0 -> 656.7 mm
- net /RCLK: track 74.8 -> 80.3 mm
- net /expr2: track 149.9 -> 155.3 mm
- net /SDA: track 446.3 -> 441.2 mm
- net /SCLK: track 69.9 -> 75.0 mm
- net /SwitchMatrix/Out15: track 167.0 -> 171.8 mm
- net /MOSI: track 72.2 -> 76.9 mm
- net /SCL: track 443.2 -> 447.0 mm, vias 9 -> 8
- net /VDD_5V0: track 375.6 -> 379.1 mm, vias 14 -> 16
- net /I2C_Reset: track 423.7 -> 420.2 mm
- net /VDD_3V3: track 622.2 -> 618.8 mm
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Other:
- board text removed: "In"
- board text removed: "Out1"
- board text removed: "Out2"
- board text removed: "R1"
- board text removed: "R2"
- board text removed: "R3"
- board text removed: "R4"
- board text removed: "R5"
- board text removed: "R6"
- board text removed: "R7"
- board text removed: "R8"
- board text removed: "R9"
- board text removed: "S1"
- board text removed: "S2"
- board text removed: "S3"
- board text removed: "S4"
- board text removed: "S5"
- board text removed: "S9"
- board text removed: "Tuner"

Commit message: Changed main to 8 loop version. Might add buffers later
Parts:
- removed H2: MountingHole, MountingHole:MountingHole_3.2mm_M3
- removed J_Return1, J_Return2, J_Send1, J_Send2: ACJS-MV-5, SamacSys_Parts:ACJSMV5
- added R69: 1k, Resistor_SMD:R_1206_3216Metric_Pad1.30x1.75mm_HandSolder, F.Cu at (185.8, 181.6)
- added R70: 1k, Resistor_SMD:R_1206_3216Metric_Pad1.30x1.75mm_HandSolder, F.Cu at (182.0, 181.6)
- C31: value 1u -> 10u
- C_Spl3, C_Spl6, C_Spl7, C_Spl8: moved to F.Cu
- PS1: value TBA_1-0310 -> QS4A_0303S1.5UP; footprint SamacSys_Parts:TBA1 -> SamacSys_Parts:QS4A_1.5UP
- R67: value 100k -> 10k
- moved H1 56.9 mm to (350.9, 162.1)
- moved C16 40.0 mm to (70.9, 142.3)
- moved C18 40.0 mm to (80.8, 156.1)
- moved J_1 40.0 mm to (70.0, 173.5)
- moved J_2 40.0 mm to (70.0, 153.5)
- moved U13 40.0 mm to (77.9, 150.9)
- moved C17 40.0 mm to (75.3, 156.1)
- moved C21 40.0 mm to (61.6, 184.0)
- moved IC21 40.0 mm to (78.0, 161.4)
- moved U14 40.0 mm to (77.7, 180.4)
- moved R42 40.0 mm to (76.6, 145.7)
- moved R43 40.0 mm to (76.6, 142.2)
- moved R44 40.0 mm to (76.6, 138.9)
- moved C_Spl8 28.6 mm to (383.0, 145.3), turned to -90 degrees
- moved C_Spl7 27.7 mm to (383.0, 150.3)
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Connections:
- net /return1 renamed /SwitchMatrix/In2
- net /return2 renamed /SwitchMatrix/In3
- net /send1 renamed /SwitchMatrix/Out1
- net /send2 renamed /SwitchMatrix/Out2
- U14 pad 10: /LoopJacks/send2_con -> unconnected-(U14-Pad10)
- U14 pad 11: /LoopJacks/return2_con -> unconnected-(U14-Pad11)
- U14 pad 8: /LoopJacks/send1_con -> unconnected-(U14-Pad8)
- U14 pad 9: /LoopJacks/return1_con -> unconnected-(U14-Pad9)
Routing:
- net /SwitchMatrix/In2: track 324.4 -> 22.0 mm, vias 2 -> 1
- net /SwitchMatrix/In3: track 301.9 -> 21.4 mm
- net /SwitchMatrix/Out1: track 344.8 -> 168.2 mm, vias 2 -> 1
- net /SwitchMatrix/Out2: track 327.0 -> 171.1 mm, vias 2 -> 1
- net /SCL: track 447.0 -> 385.6 mm, vias 8 -> 10
- net /INT: track 462.8 -> 404.7 mm, vias 2 -> 4
- net /LoopJacks/return2_con: track 54.2 -> 0.00 mm, vias 1 -> 0
- net /I2C_Reset: track 420.2 -> 366.6 mm, vias 12 -> 14
- net /VDD_15V0: track 673.7 -> 622.1 mm, vias 21 -> 23
- net /SDA: track 441.2 -> 389.9 mm, vias 9 -> 10
- net /VDD_3V3: track 618.8 -> 572.7 mm, vias 16 -> 14
- net /LoopJacks/return1_con: track 41.5 -> 0.00 mm, vias 1 -> 0
- net /LoopJacks/send2_con: track 40.6 -> 0.00 mm, vias 1 -> 0
- net /in: track 358.7 -> 318.3 mm
- net /Tuner: track 341.4 -> 301.4 mm
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Other:
- board size 392 x 61.8 mm -> 340 x 61.8 mm
