File: ControllerMainV2/Input.kicad_sch (KiCad schematic)
At the start: 12 parts, among them IC21 TMUX6112PWR, J25 Conn_01x02, U13 TL072

Commit message: Added libs
Parts:
- removed J25: Conn_01x02, symbol Connector_Generic:Conn_01x02
- J24: value (none) -> Conn_01x02; footprint (none) -> Connector_PinSocket_2.54mm:PinSocket_1x02_P2.54mm_Vertical
Other:
- moved on the sheet: C17, C18, J24, J_1

Commit message: 3D models and fixed pcbs
Parts:
- removed J24: Conn_01x02, Connector_PinSocket_2.54mm:PinSocket_1x02_P2.54mm_Vertical, symbol Connector_Generic:Conn_01x02
Changed lines of the file:
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@@
   (junction (at 100.33 34.29) (diameter 0) (color 0 0 0 0)
   )
-  (junction (at 77.978 29.21) (diameter 0) (color 0 0 0 0)
-  )
   (junction (at 100.33 41.91) (diameter 0) (color 0 0 0 0)
   )
@@
   )
   (junction (at 138.43 31.75) (diameter 0) (color 0 0 0 0)
-  )
-  (junction (at 68.961 31.75) (diameter 0) (color 0 0 0 0)
   )
   (junction (at 100.33 39.37) (diameter 0) (color 0 0 0 0)
@@
     (stroke (width 0) (type default) (color 0 0 0 0))
   )
-  (wire (pts (xy 77.978 26.67) (xy 77.978 29.21))
-    (stroke (width 0) (type default) (color 0 0 0 0))
-  )
   (wire (pts (xy 138.43 31.75) (xy 138.43 29.21))
     (stroke (width 0) (type default) (color 0 0 0 0))
@@
     (stroke (width 0) (type default) (color 0 0 0 0))
   )
-  (wire (pts (xy 77.978 29.21) (xy 81.026 29.21))
-    (stroke (width 0) (type default) (color 0 0 0 0))
-  )
   (wire (pts (xy 215.9 46.99) (xy 215.9 44.45))
     (stroke (width 0) (type default) (color 0 0 0 0))
@@
     (stroke (width 0) (type default) (color 0 0 0 0))
   )
-  (wire (pts (xy 63.881 29.21) (xy 77.978 29.21))
+  (wire (pts (xy 63.881 29.21) (xy 81.026 29.21))
     (stroke (width 0) (type default) (color 0 0 0 0))
   )
@@
     (stroke (width 0) (type default) (color 0 0 0 0))
   )
-  (wire (pts (xy 86.741 26.67) (xy 77.978 26.67))
-    (stroke (width 0) (type default) (color 0 0 0 0))
-  )
   (wire (pts (xy 100.33 46.99) (xy 100.33 44.45))
     (stroke (width 0) (type default) (color 0 0 0 0))
@@
     (stroke (width 0) (type default) (color 0 0 0 0))
   )
-  (wire (pts (xy 86.741 31.75) (xy 68.961 31.75))
-    (stroke (width 0) (type default) (color 0 0 0 0))
-  )
   (wire (pts (xy 171.45 55.88) (xy 190.5 55.88))
     (stroke (width 0) (type default) (color 0 0 0 0))
@@
   )
   (wire (pts (xy 173.99 46.99) (xy 171.45 46.99))
-    (stroke (width 0) (type default) (color 0 0 0 0))
-  )
-  (wire (pts (xy 86.741 29.21) (xy 86.741 31.75))
     (stroke (width 0) (type default) (color 0 0 0 0))
   )
@@
     (pin "5")
   )
-  (symbol (lib_id "Connector_Generic:Conn_01x02") (at 91.821 29.21 0) (mirror x) (unit 1)
-    (in_bom yes) (on_board yes) (fields_autoplaced)
-    (property "Reference" "J24" (id 0) (at 91.821 21.7002 0))
-    (property "Value" "Conn_01x02" (id 1) (at 91.821 24.2371 0))
-    (property "Footprint" "Connector_PinSocket_2.54mm:PinSocket_1x02_P2.54mm_Vertical" (id 2) (at 91.821 29.21 0)
-      (effects (font (size 1.27 1.27)) hide)
-    )
-    (property "Datasheet" "~" (id 3) (at 91.821 29.21 0)
-      (effects (font (size 1.27 1.27)) hide)
-    )
-    (pin "1")
-    (pin "2")
-  )
   (symbol (lib_id "power:GND") (at 100.33 48.26 0) (unit 1)
