File: ControllerMainV2/LoopJacks.kicad_sch (KiCad schematic)
At the start: 56 parts, among them J10 Conn_01x02, J11 Conn_01x02, J12 Conn_01x02, J13 Conn_01x02, J14 Conn_01x02, J15 Conn_01x02, J16 Conn_01x02, J17 Conn_01x02, J18 Conn_01x02, J19 Conn_01x02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

Commit message: Added libs
Parts:
- removed J10, J11, J12, J13, J14, J15, J16, J17, J18, J19, J20, J21, J22, J23, J5, J6, J7, J8, J9: Conn_01x02, symbol Connector_Generic:Conn_01x02
- removed J4: (no value), symbol Connector_Generic:Conn_01x02
Connections:
- net Addr6: now reaches R59.2, R60.1
- net Addr7: now reaches R60.2, R61.1
Other:
- moved on the sheet: J_Send1, J_Send10, J_Send2, J_Send3, J_Send4, J_Send5, J_Send6, J_Send7, J_Send8, J_Send9

Commit message: Changed main to 8 loop version. Might add buffers later
Parts:
- removed J_Return1, J_Return2, J_Send1, J_Send2: ACJS-MV-5, SamacSys_Parts:ACJSMV5, symbol Aphenol:ACJS-MV-5
Connections:
- net return1_con: no longer names the net of U14.9 (GP1)
- net return2_con: no longer names the net of U14.11 (GP3)
- net send1_con: no longer names the net of U14.8 (GP0)
- net send2_con: no longer names the net of U14.10 (GP2)
- no-connect marks 49 -> 45
