File: Status/StatusPCB/StatusPCB.kicad_sch (KiCad schematic)
At the start: 119 parts, among them Q1 BC847, Q10 BC847, Q11 2N7002, Q12 2N7002, Q13 2N7002, Q14 2N7002, Q15 2N7002, Q16 2N7002, Q17 2N7002, Q18 2N7002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

Commit message: 3D models and fixed pcbs
Parts:
- J1: value (none) -> Conn_01x08; footprint (none) -> Connector_JST:JST_PH_B8B-PH-K_1x08_P2.00mm_Vertical
- R2: value (none) -> 10k
- R3: value (none) -> 20k
- U1, U2, U3: footprint (none) -> SOIC127P1030X265-18N
