File: SwitchPCB/switchpcb_v2_left/switchpcb_v2_left.kicad_pcb (KiCad board)
At the start: 2 copper layers, 261 x 27 mm, 77 parts, among them J1 Conn_01x08, Q1 2N7002, Q10 2N7002, Q11 BC847, Q12 2N7002, Q13 BC847, Q14 2N7002, Q15 BC847, Q16 2N7002, Q17 BC847, Q18 BC847, Q19 2N7002, Q2 2N7002, Q20 2N7002, Q21 BC847, Q22 BC847, Q23 2N7002, Q24 2N7002, Q3 BC847, Q4 BC847, Q5 BC847, Q6 2N7002, Q7 BC847, Q8 2N7002, Q9 BC847, SW1 Lehle_Switch, SW2 Lehle_Switch, SW3 Lehle_Switch, SW4 Lehle_Switch, U1 74HC595, U2 74HC595

Commit message: Changed switch pcb left to 9V led supply
Parts:
- J_Main1: value Conn_01x08 -> Conn_01x09; footprint Connector_JST:JST_PH_B8B-PH-K_1x08_P2.00mm_Vertical -> Connector_JST:JST_PH_B9B-PH-K_1x09_P2.00mm_Vertical
- moved R1 2.30 mm to (150.2, 79.6)
Connections:
- D_Bl1 pad 2: /VDD3V3 -> /VDD9V0
- D_Bl2 pad 2: /VDD3V3 -> /VDD9V0
- D_Bl3 pad 2: /VDD3V3 -> /VDD9V0
- D_Bl4 pad 2: /VDD3V3 -> /VDD9V0
- D_Ge1 pad 2: /VDD3V3 -> /VDD9V0
- D_Ge2 pad 2: /VDD3V3 -> /VDD9V0
- D_Ge3 pad 2: /VDD3V3 -> /VDD9V0
- D_Ge4 pad 2: /VDD3V3 -> /VDD9V0
- J1 pad 1: /VDD3V3 -> /VDD9V0
Routing:
- net /VDD9V0: track 0.00 -> 351.4 mm, vias 0 -> 13
- net /VDD3V3: track 464.1 -> 270.9 mm, vias 6 -> 5
- net GND: track 566.3 -> 553.9 mm
- net Net-(Q3-Pad2): track 3.95 -> 6.33 mm
- net Net-(Q1-Pad3): track 4.25 -> 6.44 mm
- net /sw6: track 104.9 -> 106.9 mm
- net /On_5: track 24.8 -> 22.9 mm
- net /Stomp_4: track 67.6 -> 68.9 mm
- net /On_4: track 74.2 -> 75.4 mm
- net /Vref_blue: track 297.2 -> 296.1 mm
- net /sw5: track 109.3 -> 108.3 mm
- net Net-(Q22-Pad3): track 33.7 -> 32.9 mm
- net /sw3: track 41.3 -> 40.5 mm
- net /Vref_green: track 300.4 -> 301.0 mm
- net /On_1: track 99.8 -> 99.2 mm

Commit message: 3D models and fixed pcbs
Parts:
- SW1: moved to F.Cu
- turned SW1 to 0 degrees
Other:
- outline, holes or cut-outs redrawn

Commit message: Changed switch left to 3 switches
Parts:
- removed D_Bl1, D_Ge1: LED, LED_THT:LED_D3.0mm
- removed J_SW1: Conn_01x02, Connector_JST:JST_PH_B2B-PH-K_1x02_P2.00mm_Vertical
- removed Q1, Q2: 2N7002, Package_TO_SOT_SMD:SOT-23
- removed Q3, Q4: BC847, Package_TO_SOT_SMD:SOT-23
- removed R1, R2: 330, Resistor_SMD:R_1206_3216Metric_Pad1.30x1.75mm_HandSolder
- removed R3, R4, R5: 100k, Resistor_SMD:R_1206_3216Metric_Pad1.30x1.75mm_HandSolder
- removed SW1: Lehle_Switch, KiCad_Libs:LehleSwitch
- moved J_Main1 65.5 mm to (234.8, 96.0)
- moved R10 10.3 mm to (189.2, 80.5), turned to 180 degrees
- moved Q8 7.98 mm to (220.1, 87.7), turned to 0 degrees
- moved J_SW2 2.70 mm to (188.7, 86.0)
- moved R9 1.08 mm to (225.1, 88.9)
- moved R8 0.93 mm to (230.9, 91.5), turned to 0 degrees
- moved R13 0.83 mm to (317.9, 93.2)
Connections:
- J_Main2 pad 1: /sw1 -> /VDD3V3
Routing:
- net GND: track 553.9 -> 356.8 mm, vias 43 -> 33
- net /sw1: track 146.5 -> 0.00 mm, vias 2 -> 0
- net /Stomp_1: track 102.0 -> 0.00 mm, vias 3 -> 0
- net /VDD9V0: track 351.4 -> 250.6 mm, vias 13 -> 11
- net /On_1: track 99.2 -> 0.00 mm, vias 3 -> 0
- net /Vref_green: track 301.0 -> 204.3 mm, vias 12 -> 10
- net /SRCLK: track 191.8 -> 108.6 mm, vias 9 -> 5
- net /RCLK: track 194.8 -> 115.1 mm, vias 4 -> 2
- net /SRCLR: track 174.3 -> 97.2 mm, vias 8 -> 5
- net /Vref_blue: track 296.1 -> 226.4 mm
- net /SER: track 125.7 -> 56.9 mm, vias 6 -> 3
- net /VDD3V3: track 270.9 -> 219.3 mm
- net /sw2: track 105.4 -> 81.2 mm
- net Net-(D_Ge1-Pad1): track 8.22 -> 0.00 mm
- net /Stomp_2: track 17.8 -> 25.5 mm
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Other:
- board size 261 x 27 mm -> 187 x 27 mm
