File: PSU_Prozessor/PSU_Prozessor.kicad_sch (KiCad schematic)
At the start: 88 parts, among them IC1 6N138S, J1 ACJS-MHOP, J2 Conn_01x06, J3 FC68148S, J4 USB2066-05-RBHM-15-STB-00-01-A, J7 USB2066-05-RBHM-15-STB-00-01-A, Q1 BC847, Q2 2N7002, Q3 BC847, Q4 2N7002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

Commit message: Main schematic was not saved
Parts:
- D2: footprint Diode_THT:D_DO-35_SOD27_P7.62mm_Horizontal -> Diode_SMD:D_SOD-123
Changed lines of the file:
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@@
       (effects (font (size 1.27 1.27)) (justify left))
     )
-    (property "Footprint" "Diode_THT:D_DO-35_SOD27_P7.62mm_Horizontal" (id 2) (at 211.455 110.49 0)
+    (property "Footprint" "Diode_SMD:D_SOD-123" (id 2) (at 211.455 110.49 0)
       (effects (font (size 1.27 1.27)) hide)
     )
@@
     )
     (path "/03766177-b5de-46e5-80e8-ad9d0fb1ea03"
-      (reference "D2") (unit 1) (value "1N4148") (footprint "Diode_THT:D_DO-35_SOD27_P7.62mm_Horizontal")
+      (reference "D2") (unit 1) (value "1N4148") (footprint "Diode_SMD:D_SOD-123")
     )
     (path "/9c3666ff-48f7-42fc-87ea-b19fd9bff60f"
