File: pcb/SwitchPCB/switchpcb_v2_left/switchpcb_v2_left.kicad_sch (KiCad schematic)
At the start: 64 parts, among them J1 Conn_01x08, Q10 2N7002, Q11 BC847, Q12 2N7002, Q13 BC847, Q14 2N7002, Q15 BC847, Q16 2N7002, Q17 BC847, Q18 BC847, Q19 2N7002, Q20 2N7002, Q21 BC847, Q22 BC847, Q23 2N7002, Q24 2N7002, Q5 BC847, Q6 2N7002, Q7 BC847, Q8 2N7002, Q9 BC847, SW2 Lehle_Switch, SW3 Lehle_Switch, SW4 Lehle_Switch, U1 74HC595, U2 74HC595

Commit message: New switch pcb version with IO expander
Parts:
- removed C2: 100n, Capacitor_SMD:C_1206_3216Metric_Pad1.33x1.80mm_HandSolder, symbol Device:C
- removed J_Main2: Conn_01x08, Connector_JST:JST_PH_B8B-PH-K_1x08_P2.00mm_Vertical, symbol Connector_Generic:Conn_01x08
- removed R13, R16, R18, R24, R25, R29, R30, R6, R8: 100k, Resistor_SMD:R_1206_3216Metric_Pad1.30x1.75mm_HandSolder, symbol Device:R
- removed U1, U2: 74HC595, SamacSys_Parts:SOIC127P600X175-16N, symbol 74xx:74HC595
- added R10, R12: 10k, Resistor_SMD:R_0805_2012Metric_Pad1.20x1.40mm_HandSolder, symbol Device:R
- added U1: MCP23017_SO, Package_SO:SOIC-28W_7.5x17.9mm_P1.27mm, symbol Interface_Expansion:MCP23017_SO
- R1: renamed from R26; footprint Resistor_SMD:R_1206_3216Metric_Pad1.30x1.75mm_HandSolder -> Resistor_SMD:R_0805_2012Metric_Pad1.20x1.40mm_HandSolder
- R11: value 100k -> 10k; footprint Resistor_SMD:R_1206_3216Metric_Pad1.30x1.75mm_HandSolder -> Resistor_SMD:R_0805_2012Metric_Pad1.20x1.40mm_HandSolder
- R13: renamed from R12; footprint Resistor_SMD:R_1206_3216Metric_Pad1.30x1.75mm_HandSolder -> Resistor_SMD:R_0805_2012Metric_Pad1.20x1.40mm_HandSolder
- R14, R15, R7: footprint Resistor_SMD:R_1206_3216Metric_Pad1.30x1.75mm_HandSolder -> Resistor_SMD:R_0805_2012Metric_Pad1.20x1.40mm_HandSolder
- R16: renamed from R17; footprint Resistor_SMD:R_1206_3216Metric_Pad1.30x1.75mm_HandSolder -> Resistor_SMD:R_0805_2012Metric_Pad1.20x1.40mm_HandSolder
- R17: renamed from R19; footprint Resistor_SMD:R_1206_3216Metric_Pad1.30x1.75mm_HandSolder -> Resistor_SMD:R_0805_2012Metric_Pad1.20x1.40mm_HandSolder
- R18: renamed from R20; footprint Resistor_SMD:R_1206_3216Metric_Pad1.30x1.75mm_HandSolder -> Resistor_SMD:R_0805_2012Metric_Pad1.20x1.40mm_HandSolder
- R2: renamed from R21; footprint Resistor_SMD:R_1206_3216Metric_Pad1.30x1.75mm_HandSolder -> Resistor_SMD:R_0805_2012Metric_Pad1.20x1.40mm_HandSolder
- R3: renamed from R22; footprint Resistor_SMD:R_1206_3216Metric_Pad1.30x1.75mm_HandSolder -> Resistor_SMD:R_0805_2012Metric_Pad1.20x1.40mm_HandSolder
- R4: renamed from R27; footprint Resistor_SMD:R_1206_3216Metric_Pad1.30x1.75mm_HandSolder -> Resistor_SMD:R_0805_2012Metric_Pad1.20x1.40mm_HandSolder
- R5: renamed from R23; footprint Resistor_SMD:R_1206_3216Metric_Pad1.30x1.75mm_HandSolder -> Resistor_SMD:R_0805_2012Metric_Pad1.20x1.40mm_HandSolder
- R6: renamed from R28; footprint Resistor_SMD:R_1206_3216Metric_Pad1.30x1.75mm_HandSolder -> Resistor_SMD:R_0805_2012Metric_Pad1.20x1.40mm_HandSolder
- R8: renamed from R9; footprint Resistor_SMD:R_1206_3216Metric_Pad1.30x1.75mm_HandSolder -> Resistor_SMD:R_0805_2012Metric_Pad1.20x1.40mm_HandSolder
- R9: renamed from R10; footprint Resistor_SMD:R_1206_3216Metric_Pad1.30x1.75mm_HandSolder -> Resistor_SMD:R_0805_2012Metric_Pad1.20x1.40mm_HandSolder
- renumbered D_Bl2 to D_Bl1, D_Bl3 to D_Bl2, D_Bl4 to D_Bl3, D_Ge2 to D_Ge1, D_Ge3 to D_Ge2, D_Ge4 to D_Ge3, J_SW2 to J_SW1, J_SW3 to J_SW2, J_SW4 to J_SW3, Q17 to Q1, Q6 to Q10, Q7 to Q11, Q8 to Q12, Q9 to Q13, Q10 to Q14, Q11 to Q15, Q12 to Q16, Q13 to Q17, Q14 to Q18, Q15 to Q19, Q19 to Q2, Q16 to Q20, Q21 to Q3, Q23 to Q4, Q18 to Q5, Q20 to Q6, Q22 to Q7, Q24 to Q8, Q5 to Q9, SW2 to SW1, SW3 to SW2, SW4 to SW3
Connections:
- net GND: now also R12.2, U1.10 (VSS); no longer R11.2
- net On_2: now also U1.1 (GPB0)
- net On_3: now also U1.3 (GPB2); no longer R11.1
- net On_4: now also U1.5 (GPB4)
- net On_5: now also U1.7 (GPB6)
- net On_6: now also U1.21 (GPA0)
- net Stomp_2: now also U1.2 (GPB1)
- net Stomp_3: now also U1.4 (GPB3)
- net Stomp_4: now also U1.6 (GPB5)
- net Stomp_5: now also U1.8 (GPB7)
- net Stomp_6: now also U1.22 (GPA1)
- net VDD3V3: now also R11.1, R10.1, U1.9 (VDD)
- net sw2: now also U1.23 (GPA2)
- net sw3: now also U1.24 (GPA3)
- net sw4: now also U1.25 (GPA4)
- net sw5: now also U1.26 (GPA5)
- net sw6: now also U1.27 (GPA6)
- net RCLK renamed RESET_N
- net RESET_N: now also U1.18 (~{RESET})
- net SER renamed SCK
- net SCK: now also U1.12 (SCK)
- net SRCLK renamed SDA
- net SDA: now also U1.13 (SDA)
- net SRCLR renamed INT
- net INT: now also U1.19 (INTB), U1.20 (INTA)
- new net: R10.2, U1.16 (A1), U1.17 (A2)
- new net: R11.2, R12.1, U1.15 (A0)
- no-connect marks 4 -> 1
Other:
- moved on the sheet: J_Main1
