File: pcb/ControllerMainV2/LoopJacks.kicad_sch (KiCad schematic)
At the start: 32 parts, among them U14 MCP23009-E_SO, U15 MCP23009-E_SO, U16 MCP23009-E_SO

Commit message: New version with smaller enclosure
Parts:
- removed C21, C23: 100n, Capacitor_SMD:C_1206_3216Metric_Pad1.33x1.80mm_HandSolder, symbol Device:C
- removed J_Return10, J_Return9, J_Send10, J_Send9: ACJS-MV-5, SamacSys_Parts:ACJSMV5, symbol Aphenol:ACJS-MV-5
- removed R45, R61: 10k, Resistor_SMD:R_1206_3216Metric_Pad1.30x1.75mm_HandSolder, symbol Device:R
- removed R46, R47, R56, R57, R58, R59, R60: 20k, Resistor_SMD:R_1206_3216Metric_Pad1.30x1.75mm_HandSolder, symbol Device:R
- removed U14, U15, U16: MCP23009-E_SO, SamacSys_Parts:SOIC127P1030X265-18N, symbol SamacSys_Parts:MCP23009-E_SO
- added R10: 10k, Resistor_SMD:R_0805_2012Metric_Pad1.20x1.40mm_HandSolder, symbol Device:R
- added U2: MCP23017_SS, Package_SO:SSOP-28_5.3x10.2mm_P0.65mm, symbol Interface_Expansion:MCP23017_SS
- R9: renamed from R48; footprint Resistor_SMD:R_1206_3216Metric_Pad1.30x1.75mm_HandSolder -> Resistor_SMD:R_0805_2012Metric_Pad1.20x1.40mm_HandSolder
- renumbered C22 to C6, J_Return3 to J_Return1, J_Return4 to J_Return2, J_Return5 to J_Return3, J_Return6 to J_Return4, J_Return7 to J_Return5, J_Return8 to J_Return6, J_Send3 to J_Send1, J_Send4 to J_Send2, J_Send5 to J_Send3, J_Send6 to J_Send4, J_Send7 to J_Send5, J_Send8 to J_Send6
Connections:
- net GND: now also R10.2, U2.10 (VSS)
- net I2C_Reset: now also U2.18 (~{RESET})
- net INT: now also U2.19 (INTB), U2.20 (INTA)
- net SCL: now also U2.12 (SCK)
- net SDA: now also U2.13 (SDA)
- net VDD_3V3: now also U2.9 (VDD)
- net expr1_con: now also U2.27 (GPA6)
- net return3_con: now also U2.2 (GPB1)
- net return4_con: now also U2.4 (GPB3)
- net return5_con: now also U2.6 (GPB5)
- net return6_con: now also U2.8 (GPB7)
- net return7_con: now also U2.22 (GPA1)
- net return8_con: now also U2.24 (GPA3)
- net send3_con: now also U2.1 (GPB0)
- net send4_con: now also U2.3 (GPB2)
- net send5_con: now also U2.5 (GPB4)
- net send6_con: now also U2.7 (GPB6)
- net send7_con: now also U2.21 (GPA0)
- net send8_con: now also U2.23 (GPA2)
- new net: R10.1, U2.15 (A0), U2.16 (A1), U2.17 (A2)
- no-connect marks 45 -> 27
Other:
- moved on the sheet: C6, R9
