File: pcb/ControllerMainV2/SwitchMatrix.kicad_sch (KiCad schematic)
At the start: 18 parts, among them IC1 1462039-4, IC2 TXU0104PWR, IC3 AD75019JPZ, J3 Conn_02x08_Odd_Even, J4 Conn_02x08_Odd_Even, Q6 2N7002

Commit message: New version with smaller enclosure
Parts:
- removed C19, C20: 100n, Capacitor_SMD:C_1206_3216Metric_Pad1.33x1.80mm_HandSolder, symbol Device:C
- removed J3, J4: Conn_02x08_Odd_Even, Connector_PinHeader_1.27mm:PinHeader_2x08_P1.27mm_Vertical_SMD, symbol Connector_Generic:Conn_02x08_Odd_Even
- R3: renamed from R66; footprint Resistor_SMD:R_1206_3216Metric_Pad1.30x1.75mm_HandSolder -> Resistor_SMD:R_0805_2012Metric_Pad1.20x1.40mm_HandSolder
- R4: renamed from R64; footprint Resistor_SMD:R_1206_3216Metric_Pad1.30x1.75mm_HandSolder -> Resistor_SMD:R_0805_2012Metric_Pad1.20x1.40mm_HandSolder
- R5: renamed from R63; footprint Resistor_SMD:R_1206_3216Metric_Pad1.30x1.75mm_HandSolder -> Resistor_SMD:R_0805_2012Metric_Pad1.20x1.40mm_HandSolder
- R6: renamed from R65; footprint Resistor_SMD:R_1206_3216Metric_Pad1.30x1.75mm_HandSolder -> Resistor_SMD:R_0805_2012Metric_Pad1.20x1.40mm_HandSolder
- R7: renamed from R62; footprint Resistor_SMD:R_1206_3216Metric_Pad1.30x1.75mm_HandSolder -> Resistor_SMD:R_0805_2012Metric_Pad1.20x1.40mm_HandSolder
- renumbered C26 to C4, C30 to C5, D7 to D1, D8 to D2, D6 to D3, IC2 to IC1, IC3 to IC2, IC1 to IC3, Q6 to Q1
