File: pcb/ControllerMainV2/remote.kicad_sch (KiCad schematic)
At the start: 22 parts, among them IC22 1462039-4, IC23 1462039-4, IC24 1462039-4, IC25 1462039-4, Q1 2N7002, Q2 2N7002, Q3 2N7002, Q4 2N7002

Commit message: New version with smaller enclosure
Parts:
- removed D3, D4: 1N4148, Diode_SMD:D_SOD-123, symbol Diode:1N4148
- removed IC24, IC25: 1462039-4, SamacSys_Parts:14620394, symbol SamacSys_Parts:1462039-4
- removed J_4, J_6: ACJS-MV-5, SamacSys_Parts:ACJSMV5, symbol Aphenol:ACJS-MV-5
- removed Q3, Q4: 2N7002, Package_TO_SOT_SMD:SOT-23, symbol Transistor_FET:2N7002
- removed R52, R53, R54: 100k, Resistor_SMD:R_1206_3216Metric_Pad1.30x1.75mm_HandSolder, symbol Device:R
- R57: renamed from R49; footprint Resistor_SMD:R_1206_3216Metric_Pad1.30x1.75mm_HandSolder -> Resistor_SMD:R_0805_2012Metric_Pad1.20x1.40mm_HandSolder
- R58: renamed from R50; footprint Resistor_SMD:R_1206_3216Metric_Pad1.30x1.75mm_HandSolder -> Resistor_SMD:R_0805_2012Metric_Pad1.20x1.40mm_HandSolder
- R59: renamed from R51; footprint Resistor_SMD:R_1206_3216Metric_Pad1.30x1.75mm_HandSolder -> Resistor_SMD:R_0805_2012Metric_Pad1.20x1.40mm_HandSolder
- renumbered D1 to D5, D2 to D6, IC23 to IC10, IC22 to IC9, J_5 to J_4, J_3 to J_5, Q1 to Q4, Q2 to Q5
Connections:
- no-connect marks 22 -> 11
