File: pcb/ControllerMainV2/ControllerMainV2.kicad_pcb (KiCad board)
At the start: 2 copper layers, 340 x 61.8 mm, 197 parts, among them IC1 1462039-4, IC17 TMUX6112PWR, IC18 TMUX6112PWR, IC19 TMUX6112PWR, IC2 TXU0104PWR, IC20 TMUX6112PWR, IC21 TMUX6112PWR, IC22 1462039-4, IC23 1462039-4, IC24 1462039-4, IC25 1462039-4, IC27 1462039-4, IC3 AD75019JPZ, IC4 AD5293BRUZ-20-RL7, IC5 AD5293BRUZ-20-RL7, J1 Conn_01x07, J2 Conn_01x10, J3 Conn_02x08_Odd_Even, J4 Conn_02x08_Odd_Even, Q1 2N7002, Q2 2N7002, Q3 2N7002, Q4 2N7002, Q5 2N7002, Q6 2N7002, Q7 EL817S1_A__TU_-F, T1 Lehle_MZ_P, U1 MCP23009-E_SO, U10 TL072, U12 TL072, U13 TL072, U14 MCP23009-E_SO, U15 MCP23009-E_SO, U16 MCP23009-E_SO, U18 TL074, U2 MCP23009-E_SO, U3 TL074, U9 TL074

Commit message: New version with smaller enclosure
Parts:
- removed C2, C24, C3, C35, C36, C39, C40: 100n, Capacitor_SMD:C_1206_3216Metric_Pad1.33x1.80mm_HandSolder
- removed C31: 10u, Capacitor_SMD:C_1206_3216Metric_Pad1.33x1.80mm_HandSolder
- removed C32, C33, C34: 1u, Capacitor_SMD:C_1206_3216Metric_Pad1.33x1.80mm_HandSolder
- removed D7, D8: 1N5818, Diode_SMD:D_SOD-123
- removed H1: MountingHole, MountingHole:MountingHole_3.2mm_M3
- removed IC17, IC18, IC19, IC20, IC21: TMUX6112PWR, SamacSys_Parts:SOP65P640X120-16N
- removed IC22, IC23, IC24, IC25, IC27: 1462039-4, SamacSys_Parts:14620394
- removed J3, J4: Conn_02x08_Odd_Even, Connector_PinHeader_1.27mm:PinHeader_2x08_P1.27mm_Vertical_SMD
- removed the J_2 at (70.0, 153.5)
- removed the J_4 at (310.0, 173.5)
- removed J_6, J_Return10, J_Return9, J_Send10, J_Send9: ACJS-MV-5, SamacSys_Parts:ACJSMV5
- removed PS1: QS4A_0303S1.5UP, SamacSys_Parts:QS4A_1.5UP
- removed Q2, Q6: 2N7002, Package_TO_SOT_SMD:SOT-23
- removed Q7: EL817S1_A__TU_-F, SamacSys_Parts:SOP254P1030X390-4N
- removed R51, R53, R55, R78, R79: 100k, Resistor_SMD:R_1206_3216Metric_Pad1.30x1.75mm_HandSolder
- removed R56: 20k, Resistor_SMD:R_1206_3216Metric_Pad1.30x1.75mm_HandSolder
- removed R68: 680, Resistor_SMD:R_1206_3216Metric_Pad1.30x1.75mm_HandSolder
- removed R69, R70: 1k, Resistor_SMD:R_1206_3216Metric_Pad1.30x1.75mm_HandSolder
- removed R71, R72, R73, R74: 2.2M, Resistor_SMD:R_1206_3216Metric_Pad1.30x1.75mm_HandSolder
- removed R75: 2.2k, Resistor_SMD:R_1206_3216Metric_Pad1.30x1.75mm_HandSolder
- removed R76, R77: 100, Resistor_SMD:R_1206_3216Metric_Pad1.30x1.75mm_HandSolder
- removed R8: 33k, Resistor_SMD:R_1206_3216Metric_Pad1.30x1.75mm_HandSolder
- removed U10, U12, U13: TL072, SamacSys_Parts:SOIC127P600X175-8N
- removed U14, U15, U16: MCP23009-E_SO, SamacSys_Parts:SOIC127P1030X265-18N
- removed U18, U9: TL074, SamacSys_Parts:SOIC127P600X175-14N
- added IC10: 1462039-4, SamacSys_Parts:14620394, B.Cu at (290.4, 168.6)
- added IC6: TMUX6112PWR, SamacSys_Parts:SOP65P640X120-16N, F.Cu at (355.3, 166.7)
- added IC7: TMUX6112PWR, SamacSys_Parts:SOP65P640X120-16N, B.Cu at (262.9, 159.8)
- added IC8: 1462039-4, SamacSys_Parts:14620394, B.Cu at (239.1, 156.9)
- added IC9: 1462039-4, SamacSys_Parts:14620394, B.Cu at (290.4, 149.6)
- added U4: TL074, SamacSys_Parts:SOIC127P600X175-14N, F.Cu at (350.9, 156.4)
- added U5: TL072, Package_SO:SOIC-8_3.9x4.9mm_P1.27mm, F.Cu at (336.9, 169.6)
- added U6: TL072, Package_SO:SOIC-8_3.9x4.9mm_P1.27mm, B.Cu at (255.6, 159.9)
- added U7: TL072, Package_SO:SOIC-8_3.9x4.9mm_P1.27mm, B.Cu at (215.9, 161.7)
- C10: value 1u -> 22n; moved to B.Cu
- C11, C15: value 1u -> 100n; moved to B.Cu
- C12, C27, C28: value 22n -> 100n; moved to B.Cu
- C13, C14, C20, C_Spl6, C_Spl7, C_Spl8, D3, D5, Q5: moved to B.Cu
- C16: value 1u -> 100n
- C17, C18, C22: value 100n -> 1u
- C19: value 100n -> 22n; moved to B.Cu
- C23: value 100n -> 2.2n; moved to B.Cu
- C25, C26: value 100n -> 22n
- C30: value 100n -> 1u; moved to B.Cu
- C5: value 2.2n -> 100n; moved to B.Cu
- C6: value 22n -> 100n
- C_Spl1, C_Spl4, T1: moved to F.Cu
- C_Spl2: value 100n -> 10u; footprint Capacitor_SMD:C_1206_3216Metric_Pad1.33x1.80mm_HandSolder -> Capacitor_SMD:C_Elec_4x5.4; moved to F.Cu
- C_Spl5: value 10u -> 100n; footprint Capacitor_SMD:C_Elec_4x5.4 -> Capacitor_SMD:C_1206_3216Metric_Pad1.33x1.80mm_HandSolder
- D1: value 1N4148 -> 1N5818
- D2: value 1N4148 -> 1N5818; moved to B.Cu
- IC1: value 1462039-4 -> TXU0104PWR; footprint SamacSys_Parts:14620394 -> SamacSys_Parts:SOP65P640X120-14N; moved to B.Cu
- IC2: value TXU0104PWR -> AD75019JPZ; footprint SamacSys_Parts:SOP65P640X120-14N -> SamacSys_Parts:69802144LF
- IC3: value AD75019JPZ -> 1462039-4; footprint SamacSys_Parts:69802144LF -> SamacSys_Parts:14620394
- IC4: value AD5293BRUZ-20-RL7 -> TMUX6112PWR; footprint SamacSys_Parts:SOP65P640X120-14N -> SamacSys_Parts:SOP65P640X120-16N; moved to B.Cu
- IC5: value AD5293BRUZ-20-RL7 -> TMUX6112PWR; footprint SamacSys_Parts:SOP65P640X120-14N -> SamacSys_Parts:SOP65P640X120-16N
- J1: value Conn_01x07 -> Conn_01x06; footprint Connector_JST:JST_PH_B7B-PH-K_1x07_P2.00mm_Vertical -> Connector_JST:JST_PH_B6B-PH-K_1x06_P2.00mm_Vertical
- J2: value Conn_01x10 -> Conn_01x08; footprint Connector_JST:JST_PH_B10B-PH-K_1x10_P2.00mm_Vertical -> Connector_JST:JST_PH_B8B-PH-K_1x08_P2.00mm_Vertical
- R1: value 33k -> 10k; footprint Resistor_SMD:R_1206_3216Metric_Pad1.30x1.75mm_HandSolder -> Resistor_SMD:R_0805_2012Metric_Pad1.20x1.40mm_HandSolder
- R10: value 100k -> 10k; footprint Resistor_SMD:R_1206_3216Metric_Pad1.30x1.75mm_HandSolder -> Resistor_SMD:R_0805_2012Metric_Pad1.20x1.40mm_HandSolder
- R11, R12, R13, R14: value 100k -> 2.2M; footprint Resistor_SMD:R_1206_3216Metric_Pad1.30x1.75mm_HandSolder -> Resistor_SMD:R_0805_2012Metric_Pad1.20x1.40mm_HandSolder; moved to F.Cu
- R15, R16, R17, R18, R62: value 100k -> 2.2M; footprint Resistor_SMD:R_1206_3216Metric_Pad1.30x1.75mm_HandSolder -> Resistor_SMD:R_0805_2012Metric_Pad1.20x1.40mm_HandSolder
- R19, R20: value 100k -> 33k; footprint Resistor_SMD:R_1206_3216Metric_Pad1.30x1.75mm_HandSolder -> Resistor_SMD:R_0805_2012Metric_Pad1.20x1.40mm_HandSolder; moved to F.Cu
- R2: value 33k -> 10k; footprint Resistor_SMD:R_1206_3216Metric_Pad1.30x1.75mm_HandSolder -> Resistor_SMD:R_0805_2012Metric_Pad1.20x1.40mm_HandSolder; moved to B.Cu
- R21: value 2.35k -> 33k; footprint Resistor_SMD:R_1206_3216Metric_Pad1.30x1.75mm_HandSolder -> Resistor_SMD:R_0805_2012Metric_Pad1.20x1.40mm_HandSolder
- R22, R23, R24, R25: value 2.2M -> 33k; footprint Resistor_SMD:R_1206_3216Metric_Pad1.30x1.75mm_HandSolder -> Resistor_SMD:R_0805_2012Metric_Pad1.20x1.40mm_HandSolder; moved to F.Cu
- R26: value 2.2M -> 33k; footprint Resistor_SMD:R_1206_3216Metric_Pad1.30x1.75mm_HandSolder -> Resistor_SMD:R_0805_2012Metric_Pad1.20x1.40mm_HandSolder
- R27, R28, R29: value 2.2M -> 100k; footprint Resistor_SMD:R_1206_3216Metric_Pad1.30x1.75mm_HandSolder -> Resistor_SMD:R_0805_2012Metric_Pad1.20x1.40mm_HandSolder
- R3, R5: value 33k -> 100k; footprint Resistor_SMD:R_1206_3216Metric_Pad1.30x1.75mm_HandSolder -> Resistor_SMD:R_0805_2012Metric_Pad1.20x1.40mm_HandSolder
- R30, R31: value 100 -> 100k; footprint Resistor_SMD:R_1206_3216Metric_Pad1.30x1.75mm_HandSolder -> Resistor_SMD:R_0805_2012Metric_Pad1.20x1.40mm_HandSolder; moved to F.Cu
- R32, R33, R36, R37, R38, R40, R41, R50, R54, R9: footprint Resistor_SMD:R_1206_3216Metric_Pad1.30x1.75mm_HandSolder -> Resistor_SMD:R_0805_2012Metric_Pad1.20x1.40mm_HandSolder
- R34, R35: value 4.7M -> 100k; footprint Resistor_SMD:R_1206_3216Metric_Pad1.30x1.75mm_HandSolder -> Resistor_SMD:R_0805_2012Metric_Pad1.20x1.40mm_HandSolder
- R39, R49: value 100k -> 100; footprint Resistor_SMD:R_1206_3216Metric_Pad1.30x1.75mm_HandSolder -> Resistor_SMD:R_0805_2012Metric_Pad1.20x1.40mm_HandSolder
- R4, R6: value 33k -> 100k; footprint Resistor_SMD:R_1206_3216Metric_Pad1.30x1.75mm_HandSolder -> Resistor_SMD:R_0805_2012Metric_Pad1.20x1.40mm_HandSolder; moved to F.Cu
- R42: value 10M -> 100k; footprint Resistor_SMD:R_1206_3216Metric_Pad1.30x1.75mm_HandSolder -> Resistor_SMD:R_0805_2012Metric_Pad1.20x1.40mm_HandSolder; moved to F.Cu
- R43: value 100 -> 4.7M; footprint Resistor_SMD:R_1206_3216Metric_Pad1.30x1.75mm_HandSolder -> Resistor_SMD:R_0805_2012Metric_Pad1.20x1.40mm_HandSolder
- R44: value 100k -> 4.7M; footprint Resistor_SMD:R_1206_3216Metric_Pad1.30x1.75mm_HandSolder -> Resistor_SMD:R_0805_2012Metric_Pad1.20x1.40mm_HandSolder
- R45: value 10k -> 100k; footprint Resistor_SMD:R_1206_3216Metric_Pad1.30x1.75mm_HandSolder -> Resistor_SMD:R_0805_2012Metric_Pad1.20x1.40mm_HandSolder; moved to B.Cu
- R46, R47, R57, R58, R59: value 20k -> 100k; footprint Resistor_SMD:R_1206_3216Metric_Pad1.30x1.75mm_HandSolder -> Resistor_SMD:R_0805_2012Metric_Pad1.20x1.40mm_HandSolder; moved to B.Cu
- R48, R66: footprint Resistor_SMD:R_1206_3216Metric_Pad1.30x1.75mm_HandSolder -> Resistor_SMD:R_0805_2012Metric_Pad1.20x1.40mm_HandSolder; moved to B.Cu
- R52: value 100k -> 2.35k; footprint Resistor_SMD:R_1206_3216Metric_Pad1.30x1.75mm_HandSolder -> Resistor_SMD:R_0805_2012Metric_Pad1.20x1.40mm_HandSolder
- R60: value 20k -> 2.2M; footprint Resistor_SMD:R_1206_3216Metric_Pad1.30x1.75mm_HandSolder -> Resistor_SMD:R_0805_2012Metric_Pad1.20x1.40mm_HandSolder; moved to B.Cu
- R61: value 10k -> 2.2M; footprint Resistor_SMD:R_1206_3216Metric_Pad1.30x1.75mm_HandSolder -> Resistor_SMD:R_0805_2012Metric_Pad1.20x1.40mm_HandSolder; moved to B.Cu
- R63: value 100k -> 2.2M; footprint Resistor_SMD:R_1206_3216Metric_Pad1.30x1.75mm_HandSolder -> Resistor_SMD:R_0805_2012Metric_Pad1.20x1.40mm_HandSolder; moved to B.Cu
- R64, R65: value 100k -> 100; footprint Resistor_SMD:R_1206_3216Metric_Pad1.30x1.75mm_HandSolder -> Resistor_SMD:R_0805_2012Metric_Pad1.20x1.40mm_HandSolder; moved to B.Cu
- R67: value 10k -> 100k; footprint Resistor_SMD:R_1206_3216Metric_Pad1.30x1.75mm_HandSolder -> Resistor_SMD:R_0805_2012Metric_Pad1.20x1.40mm_HandSolder
- R7: value 33k -> 100k; footprint Resistor_SMD:R_1206_3216Metric_Pad1.30x1.75mm_HandSolder -> Resistor_SMD:R_0805_2012Metric_Pad1.20x1.40mm_HandSolder; moved to B.Cu
- U1: value MCP23009-E_SO -> MCP23017_SS; footprint SamacSys_Parts:SOIC127P1030X265-18N -> Package_SO:SSOP-28_5.3x10.2mm_P0.65mm
- U2: value MCP23009-E_SO -> MCP23017_SS; footprint SamacSys_Parts:SOIC127P1030X265-18N -> Package_SO:SSOP-28_5.3x10.2mm_P0.65mm; moved to F.Cu
- moved R9 304.5 mm to (60.1, 154.6)
- moved R10 299.6 mm to (60.1, 157.9), turned to 180 degrees
- moved C16 283.2 mm to (353.7, 156.4), turned to 0 degrees
- moved U2 270.4 mm to (66.8, 149.1)
- moved C6 265.9 mm to (59.4, 149.9), turned to 90 degrees
- moved C17 262.0 mm to (337.2, 164.1), turned to 0 degrees
- moved R42 259.2 mm to (334.2, 174.4), turned to 180 degrees
- moved C18 257.1 mm to (337.2, 175.1), turned to 0 degrees
- moved U3 214.8 mm to (351.0, 145.6), turned to 180 degrees
- moved IC5 207.1 mm to (355.3, 173.5), turned to 180 degrees
- moved IC4 198.2 mm to (350.9, 143.4), turned to 180 degrees
- moved C21 185.7 mm to (246.3, 164.4), turned to -90 degrees
- moved R62 176.7 mm to (212.3, 165.9)
- moved R44 175.3 mm to (250.8, 158.4), turned to -90 degrees
- moved R43 171.8 mm to (247.6, 158.4), turned to -90 degrees
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- renumbered J_7 to J_1, J_8 to J_2, J_1 to J_3, J_5 to J_4, J_3 to J_5, J_Return3 to J_Return1, J_Return4 to J_Return2, J_Return5 to J_Return3, J_Return6 to J_Return4, J_Return7 to J_Return5, J_Return8 to J_Return6, J_Send3 to J_Send1, J_Send4 to J_Send2, J_Send5 to J_Send3, J_Send6 to J_Send4, J_Send7 to J_Send5, J_Send8 to J_Send6
Connections:
- C1 pad 1: /VDD_15V0 -> /VDD_3V3
- C10 pad 1: Net-(C10-Pad1) -> /SwitchMatrix/Out14
- C10 pad 2: /SwitchMatrix/In15 -> Net-(C10-Pad2)
- C11 pad 1: Net-(C11-Pad1) -> /VDD_15V0
- C11 pad 2: /SwitchMatrix/In16 -> GND
- C12 pad 1: /out2 -> GND
- C12 pad 2: Net-(C12-Pad2) -> /VSS_15V0
- C13 pad 1: GND -> /VDD_15V0
- C13 pad 2: /VDD_15V0 -> GND
- C14 pad 1: /VSS_15V0 -> GND
- C14 pad 2: GND -> /VSS_15V0
- C15 pad 1: Net-(C15-Pad1) -> /VDD_15V0
- C15 pad 2: Net-(C15-Pad2) -> GND
- C16 pad 1: Net-(C16-Pad1) -> GND
- C16 pad 2: Net-(C16-Pad2) -> /VSS_15V0
- C17 pad 1: GND -> Net-(C17-Pad1)
- C17 pad 2: /VDD_15V0 -> /SwitchMatrix/In15
- C18 pad 1: /VSS_15V0 -> Net-(C18-Pad1)
- C18 pad 2: GND -> /SwitchMatrix/In16
- C19 pad 1: /VDD_15V0 -> /out2
- C19 pad 2: GND -> Net-(C19-Pad2)
- C20 pad 1: /VSS_15V0 -> GND
- C20 pad 2: GND -> /VDD_15V0
- C21 pad 1: /VDD_3V3 -> /VSS_15V0
- C22 pad 1: /VDD_3V3 -> Net-(C22-Pad1)
- C22 pad 2: GND -> Net-(C22-Pad2)
- C23 pad 1: /VDD_3V3 -> Net-(C23-Pad1)
- C23 pad 2: GND -> Net-(C23-Pad2)
- C25 pad 1: GND -> /amp2
- C25 pad 2: /VSS_15V0 -> Net-(C25-Pad2)
- C26 pad 1: /VDD_3V3 -> /amp1
- C26 pad 2: GND -> Net-(C26-Pad2)
- C27 pad 1: /amp2 -> GND
- C27 pad 2: Net-(C27-Pad2) -> /VDD_15V0
- C28 pad 1: /amp1 -> /VSS_15V0
- C28 pad 2: Net-(C28-Pad2) -> GND
- C29 pad 2: GND -> /amp2_out
- C30 pad 1: /SwitchMatrix/VDD5V0_i -> Net-(C30-Pad1)
- C30 pad 2: GND -> /amp1_out
- C4 pad 1: GND -> /VDD_3V3
- C4 pad 2: /VSS_15V0 -> GND
- C5 pad 1: Net-(C5-Pad1) -> /SwitchMatrix/VDD5V0_i
- C5 pad 2: Net-(C5-Pad2) -> GND
- C6 pad 1: /SwitchMatrix/Out13 -> /VDD_3V3
- C6 pad 2: Net-(C6-Pad2) -> GND
- C7 pad 1: /SwitchMatrix/Out14 -> /SwitchMatrix/Out15
- C8 pad 1: /SwitchMatrix/Out15 -> /SwitchMatrix/Out16
- C9 pad 1: /SwitchMatrix/Out16 -> /SwitchMatrix/Out13
- C_Spl2 pad 1: /VSS_15V0 -> /VDD_15V0
- C_Spl3 pad 1: /VDD_3V3 -> /VSS_15V0
- C_Spl4 pad 1: /VDD_15V0 -> GND
- C_Spl4 pad 2: GND -> /VSS_15V0
- C_Spl5 pad 1: GND -> /VDD_3V3
- C_Spl5 pad 2: /VSS_15V0 -> GND
- D1 pad 1: /VDD_5V0 -> /VDD_15V0
- D1 pad 2: Net-(D1-Pad2) -> /SwitchMatrix/VDD5V0_i
- D2 pad 1: /VDD_5V0 -> GND
- D2 pad 2: Net-(D2-Pad2) -> /VSS_15V0
- IC1 pad 1: /VDD_5V0 -> /VDD_3V3
- IC1 pad 2: GND -> /SCLK
- IC1 pad 3: /SwitchMatrix/VDD5V0_i -> /MOSI
- IC1 pad 4: /VDD_5V0 -> /RCLK
- IC1 pad 5: unconnected-(IC1-Pad5) -> GND
- IC1 pad 7: unconnected-(IC1-Pad7) -> GND
- IC1 pad 8: Net-(D6-Pad2) -> /CS
- IC2 pad 1: /VDD_3V3 -> /SwitchMatrix/RCLK_i
- IC2 pad 10: unconnected-(IC2-Pad10) -> GND
- IC2 pad 11: /SwitchMatrix/RCLK_i -> GND
- IC2 pad 12: /SwitchMatrix/MOSI_i -> GND
- IC2 pad 13: /SwitchMatrix/SCLK_i -> GND
- IC2 pad 14: /SwitchMatrix/VDD5V0_i -> /return8
- IC2 pad 2: /SCLK -> /SwitchMatrix/SCLK_i
- IC2 pad 3: /MOSI -> /SwitchMatrix/MOSI_i
- IC2 pad 4: /RCLK -> /VSS_15V0
- IC2 pad 5: GND -> unconnected-(IC2-Pad5)
- IC2 pad 7: GND -> /SwitchMatrix/In16
- IC2 pad 8: /CS -> /SwitchMatrix/In15
- IC2 pad 9: unconnected-(IC2-Pad9) -> GND
- IC3 pad 1: /SwitchMatrix/RCLK_i -> /VDD_5V0
- IC3 pad 2: /SwitchMatrix/SCLK_i -> GND
- IC3 pad 3: /SwitchMatrix/MOSI_i -> /SwitchMatrix/VDD5V0_i
- IC3 pad 4: /VSS_15V0 -> /VDD_5V0
- IC3 pad 7: /SwitchMatrix/In16 -> unconnected-(IC3-Pad7)
- IC3 pad 8: /SwitchMatrix/In15 -> Net-(D3-Pad2)
- IC4 pad 1: /I2C_Reset -> /Mixer1_gain
- IC4 pad 10: /MOSI -> Net-(IC4-Pad10)
- IC4 pad 11: /SCLK -> GND
- IC4 pad 12: /CS_Amp_N -> unconnected-(IC4-Pad12)
- IC4 pad 13: Net-(IC4-Pad13) -> /VDD_15V0
- IC4 pad 14: unconnected-(IC4-Pad14) -> GND
- IC4 pad 2: /VSS_15V0 -> Net-(IC4-Pad2)
- IC4 pad 3: Net-(IC4-Pad3) -> GND
- IC4 pad 4: Net-(IC4-Pad4) -> /VSS_15V0
- IC4 pad 5: Net-(IC4-Pad5) -> GND
- IC4 pad 6: /VDD_15V0 -> GND
- IC4 pad 7: Net-(C29-Pad1) -> Net-(IC4-Pad7)
- IC4 pad 8: /VDD_3V3 -> /Mixer1_gain
- IC4 pad 9: GND -> /Mixer2_gain
- IC5 pad 1: /I2C_Reset -> /Mixer1_phi
- IC5 pad 10: Net-(IC4-Pad13) -> GND
- IC5 pad 11: /SCLK -> Net-(IC5-Pad11)
- IC5 pad 12: /CS_Amp_N -> unconnected-(IC5-Pad12)
- IC5 pad 13: unconnected-(IC5-Pad13) -> /VDD_15V0
- IC5 pad 14: unconnected-(IC5-Pad14) -> Net-(IC5-Pad11)
- IC5 pad 2: /VSS_15V0 -> Net-(IC5-Pad15)
- IC5 pad 4: Net-(IC5-Pad4) -> /VSS_15V0
- IC5 pad 5: Net-(IC5-Pad5) -> GND
- IC5 pad 6: /VDD_15V0 -> Net-(IC5-Pad3)
- IC5 pad 7: Net-(C32-Pad1) -> GND
- IC5 pad 8: /VDD_3V3 -> /Mixer1_phi_n
- IC5 pad 9: GND -> /Mixer1_phi
- J1 pad 1: /CS_Amp_N -> /VDD_15V0
- J1 pad 2: /VDD_15V0 -> /VSS_15V0
- J1 pad 3: /VSS_15V0 -> /VDD_3V3
- J1 pad 4: /VDD_3V3 -> /VDD_5V0
- J1 pad 5: /VDD_5V0 -> GND
- J1 pad 6: GND -> /I2C_Reset
- J2 pad 1: /expr2 -> /expr1
- J2 pad 2: /expr1 -> /RCLK
- J2 pad 3: /EN_SPL -> /CS
- J2 pad 4: /RCLK -> /MOSI
- J2 pad 5: /CS -> /SCLK
- J2 pad 6: /MOSI -> /SCL
- J2 pad 7: /SCLK -> /SDA
- J2 pad 8: /SCL -> /INT
- J_1 pad 4: /LoopJacks/out1_con -> unconnected-(J_1-Pad4)
- J_2 pad 1: Net-(C31-Pad1) -> Net-(IC8-Pad3)
- J_2 pad 3: Net-(C5-Pad1) -> Net-(C23-Pad1)
- J_2 pad 4: Net-(C31-Pad1) -> unconnected-(J_2-Pad4)
- J_2 pad 5: Net-(J_8-Pad5) -> unconnected-(J_2-Pad5)
- Q1 pad 1: /Ctrl1 -> /EN_SPL
- Q1 pad 3: Net-(D1-Pad2) -> Net-(D3-Pad2)
- Q3 pad 1: /Ctrl3 -> /ConnGnd
- Q3 pad 3: Net-(D3-Pad2) -> Net-(D4-Pad2)
- Q4 pad 1: /Ctrl4 -> /Ctrl1
- Q4 pad 3: Net-(D4-Pad2) -> Net-(D5-Pad2)
- Q5 pad 1: /Outputs/Conn_Gnd -> /Ctrl2
- Q5 pad 3: Net-(D5-Pad2) -> Net-(D6-Pad2)
- R1 pad 1: Net-(R1-Pad1) -> /VDD_3V3
- R10 pad 1: Net-(IC17-Pad3) -> Net-(R10-Pad1)
- R10 pad 2: Net-(R10-Pad2) -> GND
- R11 pad 1: Net-(R11-Pad1) -> /SwitchMatrix/Out15
- R11 pad 2: Net-(IC17-Pad11) -> GND
- R12 pad 1: Net-(R12-Pad1) -> /SwitchMatrix/Out16
- R12 pad 2: Net-(R12-Pad2) -> GND
- R13 pad 1: Net-(IC19-Pad3) -> /SwitchMatrix/Out13
- R13 pad 2: Net-(R12-Pad2) -> GND
- R14 pad 1: Net-(IC19-Pad11) -> /SwitchMatrix/Out14
- R14 pad 2: Net-(R14-Pad2) -> GND
- R15 pad 1: GND -> Net-(C7-Pad2)
- R15 pad 2: Net-(R10-Pad2) -> GND
- R16 pad 1: GND -> Net-(C8-Pad2)
- R16 pad 2: Net-(R12-Pad2) -> GND
- R17 pad 1: GND -> Net-(C9-Pad2)
- R17 pad 2: Net-(R11-Pad1) -> GND
- R18 pad 1: GND -> Net-(C10-Pad2)
- R18 pad 2: Net-(R14-Pad2) -> GND
- R19 pad 2: Net-(R11-Pad1) -> Net-(R19-Pad2)
- R2 pad 1: Net-(R1-Pad2) -> Net-(R2-Pad1)
- R2 pad 2: Net-(IC18-Pad7) -> GND
- R20 pad 2: Net-(R14-Pad2) -> Net-(R20-Pad2)
- R21 pad 1: Net-(C31-Pad1) -> Net-(R21-Pad1)
- R21 pad 2: Net-(C5-Pad2) -> Net-(R21-Pad2)
- R22 pad 1: /SwitchMatrix/Out13 -> Net-(R22-Pad1)
- R22 pad 2: GND -> Net-(R22-Pad2)
- R23 pad 1: /SwitchMatrix/Out14 -> Net-(R19-Pad2)
- R23 pad 2: GND -> Net-(IC4-Pad7)
- R24 pad 1: /SwitchMatrix/Out15 -> Net-(R21-Pad2)
- R24 pad 2: GND -> Net-(IC4-Pad10)
- R25 pad 1: /SwitchMatrix/Out16 -> Net-(R20-Pad2)
- R25 pad 2: GND -> Net-(IC4-Pad2)
- R26 pad 1: Net-(C6-Pad2) -> Net-(R22-Pad2)
- R26 pad 2: GND -> Net-(IC4-Pad15)
- R27 pad 1: Net-(C7-Pad2) -> Net-(R28-Pad2)
- R27 pad 2: GND -> Net-(R27-Pad2)
- R28 pad 1: Net-(C8-Pad2) -> Net-(IC5-Pad3)
- R28 pad 2: GND -> Net-(R28-Pad2)
- R29 pad 1: Net-(C9-Pad2) -> Net-(R29-Pad1)
- R29 pad 2: GND -> Net-(IC5-Pad11)
- R3 pad 1: Net-(R3-Pad1) -> /CS
- R3 pad 2: Net-(R3-Pad2) -> GND
- R30 pad 1: Net-(R19-Pad1) -> Net-(R30-Pad1)
- R30 pad 2: Net-(C10-Pad1) -> Net-(R30-Pad2)
- R31 pad 1: Net-(R20-Pad1) -> Net-(IC6-Pad3)
- R31 pad 2: Net-(C11-Pad1) -> Net-(R30-Pad2)
- R32 pad 1: /SwitchMatrix/In15 -> Net-(IC6-Pad11)
- R32 pad 2: GND -> Net-(R32-Pad2)
- R33 pad 1: /SwitchMatrix/In16 -> GND
- R33 pad 2: GND -> Net-(R28-Pad2)
- R34 pad 1: /out2 -> GND
- R34 pad 2: GND -> Net-(R30-Pad2)
- R35 pad 1: Net-(C12-Pad2) -> GND
- R35 pad 2: GND -> Net-(R29-Pad1)
- R36 pad 1: Net-(IC20-Pad3) -> GND
- R36 pad 2: Net-(R36-Pad2) -> Net-(R32-Pad2)
- R37 pad 1: Net-(R36-Pad2) -> Net-(R37-Pad1)
- R37 pad 2: GND -> Net-(R29-Pad1)
- R38 pad 1: Net-(IC20-Pad11) -> Net-(R38-Pad1)
- R38 pad 2: Net-(R38-Pad2) -> Net-(R32-Pad2)
- R39 pad 1: Net-(R39-Pad1) -> Net-(R37-Pad1)
- R39 pad 2: Net-(R38-Pad2) -> Net-(C17-Pad1)
- R4 pad 1: Net-(R3-Pad2) -> /SwitchMatrix/MOSI_i
- R4 pad 2: Net-(IC18-Pad2) -> GND
- R40 pad 1: Net-(R39-Pad1) -> Net-(R38-Pad1)
- R40 pad 2: Net-(C15-Pad1) -> Net-(C18-Pad1)
- R41 pad 1: Net-(C15-Pad2) -> /SwitchMatrix/In15
- R42 pad 1: GND -> /SwitchMatrix/In16
- R42 pad 2: Net-(IC21-Pad11) -> GND
- R43 pad 1: Net-(C16-Pad1) -> /out2
- R43 pad 2: Net-(R43-Pad2) -> GND
- R44 pad 1: GND -> Net-(C19-Pad2)
- R44 pad 2: Net-(C16-Pad2) -> GND
- R45 pad 1: GND -> Net-(IC7-Pad3)
- R46 pad 2: Net-(R46-Pad2) -> GND
- R47 pad 1: Net-(R46-Pad2) -> Net-(IC7-Pad11)
- R48 pad 1: /VDD_3V3 -> Net-(R48-Pad1)
- R48 pad 2: /INT -> Net-(R47-Pad2)
- R49 pad 1: /LoopJacks/expr1_con -> Net-(R48-Pad1)
- R49 pad 2: GND -> Net-(C22-Pad1)
- R5 pad 1: Net-(R5-Pad1) -> /SwitchMatrix/VDD5V0_i
- R5 pad 2: Net-(R5-Pad2) -> /SwitchMatrix/RCLK_i
- R50 pad 1: /Ctrl1 -> Net-(C22-Pad2)
- R52 pad 1: /Ctrl3 -> Net-(IC8-Pad3)
- R52 pad 2: GND -> Net-(C23-Pad2)
- R54 pad 1: /LoopJacks/expr2_con -> /ConnGnd
- R57 pad 1: Net-(R56-Pad2) -> /LoopJacks/expr1_con
- R57 pad 2: Net-(R57-Pad2) -> GND
- R58 pad 1: Net-(R57-Pad2) -> /Ctrl1
- R58 pad 2: Net-(R58-Pad2) -> GND
- R59 pad 1: Net-(R58-Pad2) -> /Ctrl2
- R59 pad 2: /Addr6 -> GND
- R6 pad 1: Net-(R5-Pad2) -> /SwitchMatrix/SCLK_i
- R6 pad 2: Net-(IC18-Pad10) -> GND
- R60 pad 1: /Addr6 -> /amp2
- R60 pad 2: /Addr7 -> GND
- R61 pad 1: /Addr7 -> /amp1
- R61 pad 2: /VDD_3V3 -> GND
- R62 pad 1: /EN_SPL -> Net-(C25-Pad2)
- R63 pad 1: /SwitchMatrix/VDD5V0_i -> Net-(C26-Pad2)
- R63 pad 2: /SwitchMatrix/RCLK_i -> GND
- R64 pad 1: /SwitchMatrix/MOSI_i -> Net-(R64-Pad1)
- R64 pad 2: GND -> Net-(C29-Pad1)
- R65 pad 1: /SwitchMatrix/SCLK_i -> Net-(R65-Pad1)
- R65 pad 2: GND -> Net-(C30-Pad1)
- R66 pad 1: /CS -> /amp2_out
- R67 pad 1: /VDD_3V3 -> /amp1_out
- R67 pad 2: /LoopJacks/out2_con -> GND
- R7 pad 1: Net-(R7-Pad1) -> /EN_SPL
- R7 pad 2: Net-(R7-Pad2) -> GND
- R9 pad 1: Net-(R10-Pad2) -> /VDD_3V3
- R9 pad 2: Net-(R9-Pad2) -> /INT
- T1 pad 1: Net-(C15-Pad2) -> Net-(C22-Pad2)
- T1 pad 3: Net-(C31-Pad1) -> Net-(IC8-Pad3)
- T1 pad 5: Net-(C5-Pad1) -> Net-(C23-Pad1)
- U1 pad 1: /VDD_3V3 -> /Mixer1_gain
- U1 pad 10: /Ctrl3 -> GND
- U1 pad 11: /Ctrl4 -> unconnected-(U1-Pad11)
- U1 pad 12: /Outputs/Conn_Gnd -> /SCL
- U1 pad 13: /Tuner -> /SDA
- U1 pad 15: unconnected-(U1-Pad15) -> Net-(R1-Pad2)
- U1 pad 16: unconnected-(U1-Pad16) -> Net-(R2-Pad1)
- U1 pad 17: unconnected-(U1-Pad17) -> Net-(R2-Pad1)
- U1 pad 18: GND -> /I2C_Reset
- U1 pad 2: unconnected-(U1-Pad2) -> /Mixer1_phi
- U1 pad 3: /SCL -> /Mixer1_phi_n
- U1 pad 4: /SDA -> /Mixer2_gain
- U1 pad 5: /Addr7 -> /Mixer2_phi
- U1 pad 6: /I2C_Reset -> /Mixer2_phi_n
- U1 pad 7: unconnected-(U1-Pad7) -> /Out2_phi
- U1 pad 8: /Ctrl1 -> /Out2_phi_n
- U1 pad 9: /Ctrl2 -> /VDD_3V3
- U2 pad 1: /VDD_3V3 -> /LoopJacks/send3_con
- U2 pad 10: /Mixer1_phi_n -> GND
- U2 pad 11: /Mixer2_gain -> unconnected-(U2-Pad11)
- U2 pad 12: /Mixer2_phi -> /SCL
- U2 pad 13: /Mixer2_phi_n -> /SDA
- U2 pad 14: /Out2_phi -> unconnected-(U2-Pad14)
- U2 pad 15: /Out2_phi_n -> Net-(R10-Pad1)
- U2 pad 16: unconnected-(U2-Pad16) -> Net-(R10-Pad1)
- U2 pad 17: unconnected-(U2-Pad17) -> Net-(R10-Pad1)
- U2 pad 18: GND -> /I2C_Reset
- U2 pad 2: unconnected-(U2-Pad2) -> /LoopJacks/return3_con
- U2 pad 3: /SCL -> /LoopJacks/send4_con
- U2 pad 4: /SDA -> /LoopJacks/return4_con
- U2 pad 5: /Addr6 -> /LoopJacks/send5_con
- U2 pad 6: /I2C_Reset -> /LoopJacks/return5_con
- U2 pad 7: unconnected-(U2-Pad7) -> /LoopJacks/send6_con
- U2 pad 8: /Mixer1_gain -> /LoopJacks/return6_con
- U2 pad 9: /Mixer1_phi -> /VDD_3V3
- U3 pad 1: Net-(IC4-Pad3) -> Net-(R27-Pad2)
- U3 pad 10: Net-(C27-Pad2) -> Net-(R21-Pad2)
- U3 pad 12: GND -> Net-(R22-Pad2)
- U3 pad 13: Net-(IC5-Pad4) -> Net-(IC6-Pad15)
- U3 pad 14: Net-(IC5-Pad5) -> Net-(IC6-Pad15)
- U3 pad 2: Net-(IC4-Pad3) -> Net-(R27-Pad2)
- U3 pad 3: Net-(C28-Pad2) -> Net-(R19-Pad2)
- U3 pad 5: GND -> Net-(R20-Pad2)
- U3 pad 6: Net-(IC4-Pad4) -> Net-(IC5-Pad15)
- U3 pad 7: Net-(IC4-Pad5) -> Net-(IC5-Pad15)
- U3 pad 8: Net-(IC5-Pad3) -> Net-(R30-Pad1)
- U3 pad 9: Net-(IC5-Pad3) -> Net-(R30-Pad1)
Routing:
- net /VDD_3V3: track 668.7 -> 201.7 mm, vias 23 -> 9
- net GND: track 669.9 -> 227.4 mm, vias 43 -> 26
- net /VDD_15V0: track 676.0 -> 300.4 mm, vias 27 -> 21
- net /VSS_15V0: track 661.9 -> 293.5 mm, vias 18 -> 13
- net /Tuner: track 301.4 -> 0.00 mm, vias 5 -> 0
- net /CS_Amp_N: track 298.5 -> 0.00 mm, vias 5 -> 0
- net Net-(C31-Pad1): track 279.9 -> 0.00 mm, vias 7 -> 0
- net /amp2: track 268.6 -> 12.3 mm, vias 4 -> 1
- net /amp1: track 261.8 -> 15.4 mm, vias 4 -> 1
- net /amp1_out: track 236.3 -> 5.51 mm, vias 5 -> 1
- net /LoopJacks/expr1_con: track 60.8 -> 282.5 mm, vias 1 -> 5
- net /amp2_out: track 241.6 -> 21.3 mm, vias 4 -> 1
- net /send9: track 218.6 -> 0.00 mm, vias 4 -> 0
- net /send10: track 216.5 -> 0.00 mm, vias 3 -> 0
- net /send8: track 222.4 -> 33.5 mm, vias 2 -> 0
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- added copper zone on F.Cu, net /VDD_3V3
- removed copper zone on F.Cu, net /VDD_5V0
Other:
- board size 340 x 61.8 mm -> 311 x 39 mm
- board text removed: "Controller Main Rev. 2.0"
- board text removed: "MuRo Engineering"
- board text removed: "S10"

Commit message: All drill holes added
Parts:
- moved R27 5.35 mm to (359.4, 145.4), turned to 180 degrees
- moved IC3 1.25 mm to (204.8, 147.1)
- moved R20 1.02 mm to (357.0, 141.6)
- moved R25 1.02 mm to (360.2, 141.6)
- moved C26 0.50 mm to (220.8, 169.4)
Routing:
- net Net-(R27-Pad1): track 62.4 -> 67.4 mm
- net Net-(R27-Pad2): track 11.8 -> 14.7 mm
- net /amp1: track 15.4 -> 16.8 mm
- net Net-(IC5-Pad15): track 60.4 -> 59.6 mm
- net Net-(R20-Pad2): track 6.84 -> 7.59 mm
- net Net-(D3-Pad2): track 9.22 -> 8.49 mm
- net /SwitchMatrix/VDD5V0_i: track 38.9 -> 39.6 mm
- net GND: track 227.4 -> 227.9 mm
- net Net-(C26-Pad2): track 10.8 -> 11.3 mm
Other:
- board size 311 x 39 mm -> 309.2 x 39 mm
