File: pcb/ControllerMainV2/ControllerMainV2.kicad_sch (KiCad schematic)
At the start: 13 parts, among them J1 Conn_01x07, J2 Conn_01x10, U1 MCP23009-E_SO, U2 MCP23009-E_SO

Commit message: New version with smaller enclosure
Parts:
- removed J1: Conn_01x07, Connector_JST:JST_PH_B7B-PH-K_1x07_P2.00mm_Vertical, symbol Connector_Generic:Conn_01x07
- removed J2: Conn_01x10, Connector_JST:JST_PH_B10B-PH-K_1x10_P2.00mm_Vertical, symbol Connector_Generic:Conn_01x10
- removed U1, U2: MCP23009-E_SO, SamacSys_Parts:SOIC127P1030X265-18N, symbol SamacSys_Parts:MCP23009-E_SO
- added C1: 100n, Capacitor_SMD:C_1206_3216Metric_Pad1.33x1.80mm_HandSolder, symbol Device:C
- added J1: Conn_01x06, Connector_JST:JST_PH_B6B-PH-K_1x06_P2.00mm_Vertical, symbol Connector_Generic:Conn_01x06
- added J2: Conn_01x08, Connector_JST:JST_PH_B8B-PH-K_1x08_P2.00mm_Vertical, symbol Connector_Generic:Conn_01x08
- added R1, R2: 10k, Resistor_SMD:R_0805_2012Metric_Pad1.20x1.40mm_HandSolder, symbol Device:R
- added U1: MCP23017_SS, Package_SO:SSOP-28_5.3x10.2mm_P0.65mm, symbol Interface_Expansion:MCP23017_SS
- renumbered C_Spl4 to C_Spl2, C_Spl2 to C_Spl3, C_Spl5 to C_Spl4, C_Spl3 to C_Spl5
Connections:
- net CS: now also J2.3 (Pin_3)
- net Ctrl1: now also U1.21 (GPA0)
- net Ctrl2: now also U1.22 (GPA1)
- net EN_SPL: now also U1.23 (GPA2)
- net GND: now also C1.2, J1.5 (Pin_5), R2.2, U1.10 (VSS)
- net I2C_Reset: now also J1.6 (Pin_6), U1.18 (~{RESET})
- net INT: now also J2.8 (Pin_8)
- net MOSI: now also J2.4 (Pin_4)
- net Mixer1_gain: now also U1.1 (GPB0)
- net Mixer1_phi: now also U1.2 (GPB1)
- net Mixer1_phi_n: now also U1.3 (GPB2)
- net Mixer2_gain: now also U1.4 (GPB3)
- net Mixer2_phi: now also U1.5 (GPB4)
- net Mixer2_phi_n: now also U1.6 (GPB5)
- net Out2_phi: now also U1.7 (GPB6)
- net Out2_phi_n: now also U1.8 (GPB7)
- net RCLK: now also J2.2 (Pin_2)
- net SCL: now also J2.6 (Pin_6), U1.12 (SCK)
- net SCLK: now also J2.5 (Pin_5)
- net SDA: now also J2.7 (Pin_7), U1.13 (SDA)
- net VDD_15V0: now also J1.1 (Pin_1)
- net VDD_3V3: now also C1.1, J1.3 (Pin_3), R1.1, U1.9 (VDD)
- net VDD_5V0: now also J1.4 (Pin_4)
- net VSS_15V0: now also J1.2 (Pin_2)
- net expr1: now also J2.1 (Pin_1)
- new net: R2.1, U1.16 (A1), U1.17 (A2)
- new net: R1.2, U1.15 (A0)
- new net ConnGnd: U1.24 (GPA3)
- no-connect marks 10 -> 8
Other:
- sheet Buffer ports: added none; removed CS_N, MOSI, Reset_N, SCLK, VDD_3V3
- sheet Input ports: added none; removed VDD_15V0, VSS_15V0, d_en_tuner
- sheet LoopJacks ports: added none; removed Addr6, Addr7, Return10, Return9, Send10, Send9, expr2_con, out1_con, out2_con
- sheet Outputs ports: added none; removed VDD_3V3, out1_con, out2_con
- sheet Remote ports: added none; removed Ctrl3, Ctrl4, Expr2, Expr2_con

Commit message: All drill holes added
Parts:
- removed H1: MountingHole, MountingHole:MountingHole_3.2mm_M3, symbol Mechanical:MountingHole
Changed lines of the file:
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@@
     (pin "2")
-  )
-  (symbol (lib_id "Mechanical:MountingHole") (at 127 24.13 0) (unit 1)
-    (in_bom yes) (on_board yes) (fields_autoplaced)
-    (property "Reference" "H1" (id 0) (at 129.54 23.2953 0)
-      (effects (font (size 1.27 1.27)) (justify left))
-    )
-    (property "Value" "MountingHole" (id 1) (at 129.54 25.8322 0)
-      (effects (font (size 1.27 1.27)) (justify left))
-    )
-    (property "Footprint" "MountingHole:MountingHole_3.2mm_M3" (id 2) (at 127 24.13 0)
-      (effects (font (size 1.27 1.27)) hide)
-    )
-    (property "Datasheet" "~" (id 3) (at 127 24.13 0)
-      (effects (font (size 1.27 1.27)) hide)
-    )
   )
   (symbol (lib_id "Device:C_Polarized") (at 82.55 59.69 0) (unit 1)
@@
       (reference "D6") (unit 1) (value "1N4148") (footprint "Diode_SMD:D_SOD-123")
     )
-    (path "/d7335a40-39b2-470c-8efe-04c325566c0a"
-      (reference "H1") (unit 1) (value "MountingHole") (footprint "MountingHole:MountingHole_3.2mm_M3")
-    )
     (path "/00000000-0000-0000-0000-0000618c6d5c/0d8484ee-27b7-4184-9e64-bb02806b1625"
